File: fotovoltaika/schema.sch (EAGLE design)
At the start: 16 parts, among them K1 G2R, K2 G2R, K3 G2R, K5 G2R, K7 G2R, K8 G2R

Commit message: +
Parts:
- added 12/230V2: 12/230V, trafo:EI30-1
- added 230/12V2: 230/12V, trafo:EI30-1
- added D5, D6: 1N4004, diode:1N4004
- added K4, K6, K9: G2R, relay:G2R
- added SL3: (no value), con-amp-quick:M02
Connections:
- new net N$15: 12/230V2.P2, D5.A, K42.O
- new net N$16: K61.1, K92.S
- new net N$17: 230/12V2.P1, K92.O
- new net N$18: 230/12V2.S4, D6.A
- new net N$19: K41.2, SL3.2
- new net N$20: K91.1, SL3.1
- new net N$21: 12/230V2.S3, K62.S
- net +12V: now also D5.C, D6.C, K42.P
- net +3V3: now also K41.1, K91.2
- net GND: now also 12/230V2.P1, 230/12V2.S3; no longer K11.2, K51.2
- net PE: now also 12/230V2.S4, 230/12V2.P2, K11.2, K51.2, K61.2
- net VCC: now also K62.O, K62.P, K92.P
Other:
- moved on the sheet: 12/230V1, 230/12V1, D3, D4, K5, K7, K8, SL2
