File: fotovoltaika/napeti.sch (EAGLE design)
At the start: 15 parts, among them X5 JST-XH-04-PIN-LONG-PAD

Commit message: zmena na konektory JST-XH
Parts:
- removed X1, X2, X3, X4: (no value), con-wago-500:W237-102
- added X6, X7: JST-XH-04-PIN-LONG-PAD, Rembrandt:JST-XH-04-PIN-LONG-PAD
Connections:
- net N$10: now also X6-3.S; no longer X1-2.KL
- net N$14: now also X6-1.S; no longer X2-2.KL
- net N$2: now also X6-4.S; no longer X1-1.KL
- net N$3: now also X7-3.S; no longer X3-2.KL
- net N$5: now also X6-2.S; no longer X2-1.KL
- net N$6: now also X7-1.S; no longer X4-2.KL
- net N$7: now also X7-4.S; no longer X3-1.KL
- net N$8: now also X7-2.S; no longer X4-1.KL
Changed lines of the file:
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@@
 <part name="R7" library="rcl" library_urn="urn:adsk.eagle:library:334" deviceset="R-EU_" device="0204/7" package3d_urn="urn:adsk.eagle:package:23498/1"/>
 <part name="R8" library="rcl" library_urn="urn:adsk.eagle:library:334" deviceset="R-EU_" device="0204/7" package3d_urn="urn:adsk.eagle:package:23498/1"/>
-<part name="X1" library="con-wago-500" library_urn="urn:adsk.eagle:library:195" deviceset="W237-102" device="" package3d_urn="urn:adsk.eagle:package:10688/1"/>
-<part name="X2" library="con-wago-500" library_urn="urn:adsk.eagle:library:195" deviceset="W237-102" device="" package3d_urn="urn:adsk.eagle:package:10688/1"/>
-<part name="X3" library="con-wago-500" library_urn="urn:adsk.eagle:library:195" deviceset="W237-102" device="" package3d_urn="urn:adsk.eagle:package:10688/1"/>
-<part name="X4" library="con-wago-500" library_urn="urn:adsk.eagle:library:195" deviceset="W237-102" device="" package3d_urn="urn:adsk.eagle:package:10688/1"/>
 <part name="X5" library="Rembrandt" deviceset="JST-XH-04-PIN" device="-LONG-PAD"/>
+<part name="X6" library="Rembrandt" deviceset="JST-XH-04-PIN" device="-LONG-PAD"/>
+<part name="X7" library="Rembrandt" deviceset="JST-XH-04-PIN" device="-LONG-PAD"/>
 </parts>
 <sheets>
@@
 <attribute name="VALUE" x="104.902" y="21.59" size="1.778" layer="96" rot="R90"/>
 </instance>
-<instance part="X1" gate="-1" x="25.4" y="5.08" smashed="yes" rot="R90">
-<attribute name="NAME" x="24.511" y="5.08" size="1.778" layer="95" rot="R270"/>
-</instance>
-<instance part="X1" gate="-2" x="33.02" y="5.08" smashed="yes" rot="R90">
-<attribute name="VALUE" x="36.703" y="2.54" size="1.778" layer="96" rot="R90"/>
-<attribute name="NAME" x="32.131" y="5.08" size="1.778" layer="95" rot="R270"/>
-</instance>
-<instance part="X2" gate="-1" x="45.72" y="5.08" smashed="yes" rot="R90">
-<attribute name="NAME" x="44.831" y="5.08" size="1.778" layer="95" rot="R270"/>
-</instance>
-<instance part="X2" gate="-2" x="53.34" y="5.08" smashed="yes" rot="R90">
-<attribute name="VALUE" x="57.023" y="2.54" size="1.778" layer="96" rot="R90"/>
-<attribute name="NAME" x="52.451" y="5.08" size="1.778" layer="95" rot="R270"/>
-</instance>
-<instance part="X3" gate="-1" x="73.66" y="5.08" smashed="yes" rot="R90">
-<attribute name="NAME" x="72.771" y="5.08" size="1.778" layer="95" rot="R270"/>
-</instance>
-<instance part="X3" gate="-2" x="81.28" y="5.08" smashed="yes" rot="R90">
-<attribute name="VALUE" x="84.963" y="2.54" size="1.778" layer="96" rot="R90"/>
-<attribute name="NAME" x="80.391" y="5.08" size="1.778" layer="95" rot="R270"/>
-</instance>
-<instance part="X4" gate="-1" x="93.98" y="5.08" smashed="yes" rot="R90">
-<attribute name="NAME" x="93.091" y="5.08" size="1.778" layer="95" rot="R270"/>
-</instance>
-<instance part="X4" gate="-2" x="101.6" y="5.08" smashed="yes" rot="R90">
-<attribute name="VALUE" x="105.283" y="2.54" size="1.778" layer="96" rot="R90"/>
-<attribute name="NAME" x="100.711" y="5.08" size="1.778" layer="95" rot="R270"/>
-</instance>
 <instance part="X5" gate="-1" x="45.72" y="88.9" smashed="yes" rot="R90">
 <attribute name="NAME" x="46.482" y="91.44" size="1.524" layer="95" rot="R90"/>
@@
 <instance part="X5" gate="-4" x="53.34" y="88.9" smashed="yes" rot="R90">
 <attribute name="NAME" x="54.102" y="91.44" size="1.524" layer="95" rot="R90"/>
+</instance>
+<instance part="X6" gate="-1" x="40.64" y="-7.62" smashed="yes" rot="R270">
+<attribute name="NAME" x="39.878" y="-10.16" size="1.524" layer="95" rot="R270"/>
+<attribute name="VALUE" x="42.037" y="-6.858" size="1.778" layer="96" rot="R270"/>
+</instance>
+<instance part="X6" gate="-2" x="38.1" y="-7.62" smashed="yes" rot="R270">
+<attribute name="NAME" x="37.338" y="-10.16" size="1.524" layer="95" rot="R270"/>
+</instance>
+<instance part="X6" gate="-3" x="35.56" y="-7.62" smashed="yes" rot="R270">
+<attribute name="NAME" x="34.798" y="-10.16" size="1.524" layer="95" rot="R270"/>
+</instance>
+<instance part="X6" gate="-4" x="33.02" y="-7.62" smashed="yes" rot="R270">
+<attribute name="NAME" x="32.258" y="-10.16" size="1.524" layer="95" rot="R270"/>
+</instance>
+<instance part="X7" gate="-1" x="91.44" y="-7.62" smashed="yes" rot="R270">
+<attribute name="NAME" x="90.678" y="-10.16" size="1.524" layer="95" rot="R270"/>
+<attribute name="VALUE" x="92.837" y="-6.858" size="1.778" layer="96" rot="R270"/>
+</instance>
+<instance part="X7" gate="-2" x="88.9" y="-7.62" smashed="yes" rot="R270">
+<attribute name="NAME" x="88.138" y="-10.16" size="1.524" layer="95" rot="R270"/>
+</instance>
+<instance part="X7" gate="-3" x="86.36" y="-7.62" smashed="yes" rot="R270">
+<attribute name="NAME" x="85.598" y="-10.16" size="1.524" layer="95" rot="R270"/>
+</instance>
+<instance part="X7" gate="-4" x="83.82" y="-7.62" smashed="yes" rot="R270">
+<attribute name="NAME" x="83.058" y="-10.16" size="1.524" layer="95" rot="R270"/>
 </instance>
 </instances>
@@
 <pinref part="R2" gate="G$1" pin="1"/>
 <wire x1="38.1" y1="20.32" x2="33.02" y2="20.32" width="0.1524" layer="91"/>
-<wire x1="33.02" y1="10.16" x2="33.02" y2="20.32" width="0.1524" layer="91"/>
 <junction x="33.02" y="20.32"/>
-<pinref part="X1" gate="-2" pin="KL"/>
+<wire x1="33.02" y1="20.32" x2="33.02" y2="0" width="0.1524" layer="91"/>
+<wire x1="33.02" y1="0" x2="35.56" y2="0" width="0.1524" layer="91"/>
+<pinref part="X6" gate="-3" pin="S"/>
+<wire x1="35.56" y1="0" x2="35.56" y2="-5.08" width="0.1524" layer="91"/>
 </segment>
 </net>
@@
 <pinref part="R4" gate="G$1" pin="1"/>
 <wire x1="58.42" y1="20.32" x2="53.34" y2="20.32" width="0.1524" layer="91"/>
-<wire x1="53.34" y1="10.16" x2="53.34" y2="20.32" width="0.1524" layer="91"/>
 <junction x="53.34" y="20.32"/>
 <wire x1="38.1" y1="40.64" x2="58.42" y2="40.64" width="0.1524" layer="91"/>
-<pinref part="X2" gate="-2" pin="KL"/>
+<pinref part="X6" gate="-1" pin="S"/>
+<wire x1="40.64" y1="-5.08" x2="53.34" y2="-5.08" width="0.1524" layer="91"/>
+<wire x1="53.34" y1="-5.08" x2="53.34" y2="20.32" width="0.1524" layer="91"/>
 </segment>
 </net>
@@
 <segment>
 <pinref part="R1" gate="G$1" pin="1"/>
-<wire x1="25.4" y1="20.32" x2="25.4" y2="10.16" width="0.1524" layer="91"/>
-<pinref part="X1" gate="-1" pin="KL"/>
+<wire x1="25.4" y1="20.32" x2="25.4" y2="-5.08" width="0.1524" layer="91"/>
+<pinref part="X6" gate="-4" pin="S"/>
+<wire x1="25.4" y1="-5.08" x2="33.02" y2="-5.08" width="0.1524" layer="91"/>
 </segment>
 </net>
@@
 <segment>
 <pinref part="R3" gate="G$1" pin="1"/>
-<wire x1="45.72" y1="20.32" x2="45.72" y2="10.16" width="0.1524" layer="91"/>
-<pinref part="X2" gate="-1" pin="KL"/>
+<pinref part="X6" gate="-2" pin="S"/>
+<wire x1="38.1" y1="-5.08" x2="38.1" y2="0" width="0.1524" layer="91"/>
+<wire x1="38.1" y1="0" x2="45.72" y2="0" width="0.1524" layer="91"/>
+<wire x1="45.72" y1="0" x2="45.72" y2="20.32" width="0.1524" layer="91"/>
 </segment>
 </net>
@@
 <pinref part="R6" gate="G$1" pin="1"/>
 <wire x1="86.36" y1="20.32" x2="81.28" y2="20.32" width="0.1524" layer="91"/>
-<wire x1="81.28" y1="10.16" x2="81.28" y2="20.32" width="0.1524" layer="91"/>
+<wire x1="81.28" y1="2.54" x2="81.28" y2="20.32" width="0.1524" layer="91"/>
 <junction x="81.28" y="20.32"/>
 <pinref part="ADC11150X4A" gate="G$1" pin="2"/>
 <wire x1="78.74" y1="55.88" x2="86.36" y2="55.88" width="0.1524" layer="91"/>
 <wire x1="86.36" y1="55.88" x2="86.36" y2="20.32" width="0.1524" layer="91"/>
-<pinref part="X3" gate="-2" pin="KL"/>
+<pinref part="X7" gate="-3" pin="S"/>
+<wire x1="86.36" y1="-5.08" x2="86.36" y2="2.54" width="0.1524" layer="91"/>
+<wire x1="86.36" y1="2.54" x2="81.28" y2="2.54" width="0.1524" layer="91"/>
 </segment>
 </net>
@@
 <pinref part="R8" gate="G$1" pin="1"/>
 <wire x1="106.68" y1="20.32" x2="101.6" y2="20.32" width="0.1524" layer="91"/>
-<wire x1="101.6" y1="10.16" x2="101.6" y2="20.32" width="0.1524" layer="91"/>
 <junction x="101.6" y="20.32"/>
 <pinref part="ADC11150X4A" gate="G$1" pin="4"/>
 <wire x1="78.74" y1="60.96" x2="106.68" y2="60.96" width="0.1524" layer="91"/>
 <wire x1="106.68" y1="60.96" x2="106.68" y2="20.32" width="0.1524" layer="91"/>
-<pinref part="X4" gate="-2" pin="KL"/>
+<pinref part="X7" gate="-1" pin="S"/>
+<wire x1="91.44" y1="-5.08" x2="101.6" y2="-5.08" width="0.1524" layer="91"/>
+<wire x1="101.6" y1="-5.08" x2="101.6" y2="20.32" width="0.1524" layer="91"/>
 </segment>
 </net>
@@
 <segment>
 <pinref part="R5" gate="G$1" pin="1"/>
-<wire x1="73.66" y1="20.32" x2="73.66" y2="10.16" width="0.1524" layer="91"/>
-<pinref part="X3" gate="-1" pin="KL"/>
+<pinref part="X7" gate="-4" pin="S"/>
+<wire x1="83.82" y1="-5.08" x2="73.66" y2="-5.08" width="0.1524" layer="91"/>
+<wire x1="73.66" y1="-5.08" x2="73.66" y2="20.32" width="0.1524" layer="91"/>
 </segment>
 </net>
@@
 <segment>
 <pinref part="R7" gate="G$1" pin="1"/>
-<wire x1="93.98" y1="20.32" x2="93.98" y2="10.16" width="0.1524" layer="91"/>
-<pinref part="X4" gate="-1" pin="KL"/>
-</segment>
-</net>
+<wire x1="93.98" y1="20.32" x2="93.98" y2="2.54" width="0.1524" layer="91"/>
+<pinref part="X7" gate="-2" pin="S"/>
+<wire x1="88.9" y1="-5.08" x2="88.9" y2="2.54" width="0.1524" layer="91"/>
+<wire x1="88.9" y1="2.54" x2="93.98" y2="2.54" width="0.1524" layer="91"/>
+</segment>
+</net>

Commit message: zmena delicu
Parts:
- R1: value 15k -> 10k
- R3: value 10k -> 6k8
- R4: value 4k7 -> 2k2
Changed lines of the file:
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@@
 <part name="ADC11150X4B" library="con-amp-quick" library_urn="urn:adsk.eagle:library:125" deviceset="M10" device="" package3d_urn="urn:adsk.eagle:package:5963/1"/>
 <part name="ADC11150X4A" library="con-amp-quick" library_urn="urn:adsk.eagle:library:125" deviceset="M10" device="" package3d_urn="urn:adsk.eagle:package:5963/1"/>
-<part name="R1" library="rcl" library_urn="urn:adsk.eagle:library:334" deviceset="R-EU_" device="0204/7" package3d_urn="urn:adsk.eagle:package:23498/1" value="15k"/>
+<part name="R1" library="rcl" library_urn="urn:adsk.eagle:library:334" deviceset="R-EU_" device="0204/7" package3d_urn="urn:adsk.eagle:package:23498/1" value="10k"/>
 <part name="R2" library="rcl" library_urn="urn:adsk.eagle:library:334" deviceset="R-EU_" device="0204/7" package3d_urn="urn:adsk.eagle:package:23498/1" value="4k7"/>
-<part name="R3" library="rcl" library_urn="urn:adsk.eagle:library:334" deviceset="R-EU_" device="0204/7" package3d_urn="urn:adsk.eagle:package:23498/1" value="10k"/>
-<part name="R4" library="rcl" library_urn="urn:adsk.eagle:library:334" deviceset="R-EU_" device="0204/7" package3d_urn="urn:adsk.eagle:package:23498/1" value="4k7"/>
+<part name="R3" library="rcl" library_urn="urn:adsk.eagle:library:334" deviceset="R-EU_" device="0204/7" package3d_urn="urn:adsk.eagle:package:23498/1" value="6k8"/>
+<part name="R4" library="rcl" library_urn="urn:adsk.eagle:library:334" deviceset="R-EU_" device="0204/7" package3d_urn="urn:adsk.eagle:package:23498/1" value="2k2"/>
 <part name="R5" library="rcl" library_urn="urn:adsk.eagle:library:334" deviceset="R-EU_" device="0204/7" package3d_urn="urn:adsk.eagle:package:23498/1" value="10k"/>
 <part name="R6" library="rcl" library_urn="urn:adsk.eagle:library:334" deviceset="R-EU_" device="0204/7" package3d_urn="urn:adsk.eagle:package:23498/1" value="4k7"/>

Commit message: +
Connections:
- net SCL: no longer ADC11150X4A.5
- net SDA: no longer ADC11150X4B.5
Changed lines of the file:
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@@
 <segment>
 <pinref part="ADC11150X4B" gate="G$1" pin="8"/>
-<wire x1="30.48" y1="71.12" x2="35.56" y2="71.12" width="0.1524" layer="91"/>
-<wire x1="35.56" y1="71.12" x2="50.8" y2="71.12" width="0.1524" layer="91"/>
+<wire x1="30.48" y1="71.12" x2="50.8" y2="71.12" width="0.1524" layer="91"/>
 <wire x1="50.8" y1="71.12" x2="50.8" y2="86.36" width="0.1524" layer="91"/>
 <pinref part="ADC11150X4A" gate="G$1" pin="8"/>
@@
 <junction x="50.8" y="71.12"/>
 <label x="53.34" y="99.06" size="1.778" layer="95"/>
-<pinref part="ADC11150X4B" gate="G$1" pin="5"/>
-<wire x1="30.48" y1="63.5" x2="35.56" y2="63.5" width="0.1524" layer="91"/>
-<wire x1="35.56" y1="63.5" x2="35.56" y2="71.12" width="0.1524" layer="91"/>
-<junction x="35.56" y="71.12"/>
 <pinref part="X5" gate="-3" pin="S"/>
 </segment>
@@
 <pinref part="ADC11150X4A" gate="G$1" pin="7"/>
 <wire x1="53.34" y1="73.66" x2="53.34" y2="86.36" width="0.1524" layer="91"/>
-<wire x1="78.74" y1="68.58" x2="83.82" y2="68.58" width="0.1524" layer="91"/>
-<wire x1="83.82" y1="68.58" x2="88.9" y2="68.58" width="0.1524" layer="91"/>
+<wire x1="78.74" y1="68.58" x2="88.9" y2="68.58" width="0.1524" layer="91"/>
 <wire x1="88.9" y1="68.58" x2="88.9" y2="86.36" width="0.1524" layer="91"/>
 <wire x1="88.9" y1="86.36" x2="66.04" y2="86.36" width="0.1524" layer="91"/>
@@
 <junction x="53.34" y="73.66"/>
 <label x="60.96" y="99.06" size="1.778" layer="95"/>
-<pinref part="ADC11150X4A" gate="G$1" pin="5"/>
-<wire x1="78.74" y1="63.5" x2="83.82" y2="63.5" width="0.1524" layer="91"/>
-<wire x1="83.82" y1="63.5" x2="83.82" y2="68.58" width="0.1524" layer="91"/>
-<junction x="83.82" y="68.58"/>
 <pinref part="X5" gate="-4" pin="S"/>
 </segment>
